File: M4-Shim-2.sch (EAGLE design)
At the start: 36 parts, among them SW1 KMR2, U1 ATSAMD51J, U2 2MB Flash, U3 AP2112-3.3, X1 32.768

Commit message: Add PDF of rev 2 schematic
Other:
- note added: "2"
Changed lines of the file:
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@@
 <text x="167.64" y="111.76" size="1.778" layer="97">CAN1_RX</text>
 <text x="330.2" y="27.94" size="5.08" layer="94">M4 Shim for PoE-FeatherWing</text>
+<text x="419.1" y="7.62" size="2.54" layer="94">2</text>
 </plain>
 <instances>
